Commit message: feat(genesis_ros2_control): native SystemInterface via /dev/shm seqlock
Sibling ament_cmake package implementing a native
hardware_interface::SystemInterface plugin, genesis_ros2_control::
GenesisSystem, that talks to the Python genesis_bridge through a
lock-free shared-memory region at /dev/shm/genesis_ros2_control.<robot>.

Replaces the roadmap's pybind11 in-process plan (item 13 -- Tier C)
with shared-memory IPC:
  - avoids embedding CPython inside a pluginlib-loaded .so (fragile)
  - keeps the bridge's single-writer main-thread scene.step() intact
  - crashes on either side do not take down the other
  - sub-microsecond read/write at 1 kHz+ control rates

Layout (genesis_ros2_control/include/.../shm_protocol.h):
  - GenesisShmHandshake (magic, version, n_joints, joint_name table)
  - GenesisShmState     (seqlock, stamp, position/velocity/effort arrays)
  - GenesisShmCommand   (seqlock, per-joint cmd_mask bits + pos/vel/eff)
  - cache-line padded to avoid false sharing between regions

Writer protocol: seq <- seq+1 (odd, in-progress) -> write payload ->
seq <- seq+1 (even, stable). Reader confirms seq is even, reads,
re-reads seq, retries on mismatch. No syscalls on the hot path.

Added:
- genesis_ros2_control/  ament_cmake package (package.xml, CMakeLists,
  plugin_description, src/genesis_system.cpp, include headers).
- genesis_ros/genesis_ros/control/shm_bridge.py: Python side. Dual
  GenesisPublisher + GenesisSubscriber. ctypes Structure layout
  mirrors the C header; magic + version checked on mmap.
- franka_scene.py wires register_shm_bridge(bridge, robot='franka')
  by default (GENESIS_DISABLE_SHM=1 to opt out).
- franka_panda.urdf.xacro gains a 'hardware' arg: 'shm' (default,
  genesis_ros2_control/GenesisSystem) or 'topic' (community
  topic_based_ros2_control, unchanged).
- franka.launch.py: new --hardware launch arg threads through to xacro.
- packaging/ros-jazzy-genesis-ros2-control/build.sh + build-all.sh
  hook: ships a fourth .deb (ros-jazzy-genesis-ros2-control) produced
  via bloom-generate rosdebian.

Dependencies (all stock rosdep keys):
  hardware_interface, pluginlib, rclcpp, rclcpp_lifecycle,
  controller_manager.

Not yet addressed (follow-ups):
- ROS2_INTEGRATION_PLAN.md update documenting this approach as the
  superseded version of item 13.
- Runtime verification on the devcontainer.
- Integration test that spins controller_manager against a running
  franka_demo.

File: genesis_ros/urdf/franka_panda.urdf.xacro (robot description, xacro)
@@ -14,4 +14,11 @@
   <xacro:arg name="base_urdf"
              default="/opt/genesis/assets/urdf/panda_bullet/panda.urdf"/>
+  <!--
+    hardware:
+      "shm"    genesis_ros2_control/GenesisSystem (native, /dev/shm)
+      "topic"  topic_based_ros2_control/TopicBasedSystem (community)
+  -->
+  <xacro:arg name="hardware"       default="shm"/>
+  <xacro:arg name="robot_name"     default="franka"/>
   <xacro:arg name="commands_topic" default="/franka/joint_commands"/>
   <xacro:arg name="states_topic"   default="/franka/joint_states"/>
@@ -20,26 +27,35 @@
        <robot>'s children into this one. -->
   <xacro:include filename="$(arg base_urdf)"/>
-  <!-- Helper: a single topic-based command+state joint interface. -->
-  <xacro:macro name="panda_topic_joint" params="name">
+  <!-- Helper: a single command+state joint interface used by either
+       backend. -->
+  <xacro:macro name="panda_joint_iface" params="name">
     <joint name="${name}">
       <command_interface name="position"/>
       <state_interface name="position"/>
       <state_interface name="velocity"/>
+      <state_interface name="effort"/>
     </joint>
   </xacro:macro>
-  <ros2_control name="panda_topic_bridge" type="system">
+  <ros2_control name="panda_hw" type="system">
     <hardware>
-      <plugin>topic_based_ros2_control/TopicBasedSystem</plugin>
-      <param name="joint_commands_topic">$(arg commands_topic)</param>
-      <param name="joint_states_topic">$(arg states_topic)</param>
-      <param name="sum_wrapped_joint_states">false</param>
+      <xacro:if value="${'$(arg hardware)' == 'shm'}">
+        <plugin>genesis_ros2_control/GenesisSystem</plugin>
+        <param name="robot_name">$(arg robot_name)</param>
+        <param name="wait_for_bridge_sec">10.0</param>
+      </xacro:if>
+      <xacro:if value="${'$(arg hardware)' == 'topic'}">
+        <plugin>topic_based_ros2_control/TopicBasedSystem</plugin>
+        <param name="joint_commands_topic">$(arg commands_topic)</param>
+        <param name="joint_states_topic">$(arg states_topic)</param>
+        <param name="sum_wrapped_joint_states">false</param>
+      </xacro:if>
     </hardware>
-    <xacro:panda_topic_joint name="panda_joint1"/>
-    <xacro:panda_topic_joint name="panda_joint2"/>
-    <xacro:panda_topic_joint name="panda_joint3"/>
-    <xacro:panda_topic_joint name="panda_joint4"/>
-    <xacro:panda_topic_joint name="panda_joint5"/>
-    <xacro:panda_topic_joint name="panda_joint6"/>
-    <xacro:panda_topic_joint name="panda_joint7"/>
+    <xacro:panda_joint_iface name="panda_joint1"/>
+    <xacro:panda_joint_iface name="panda_joint2"/>
+    <xacro:panda_joint_iface name="panda_joint3"/>
+    <xacro:panda_joint_iface name="panda_joint4"/>
+    <xacro:panda_joint_iface name="panda_joint5"/>
+    <xacro:panda_joint_iface name="panda_joint6"/>
+    <xacro:panda_joint_iface name="panda_joint7"/>
   </ros2_control>
 </robot>
